File: PCB/MicroMouse/main_board/motors.kicad_sch (KiCad schematic)
At the start: 3 parts, among them J2 Conn_01x06, J3 Conn_01x06, U3 TB6612FNG

Commit message: PCB prototype
Parts:
- removed J2, J3: Conn_01x06, Connector_Molex:Molex_KK-254_AE-6410-06A_1x06_P2.54mm_Vertical, symbol Connector_Generic:Conn_01x06
- added J11, J2: Conn_01x02, Connector_PinSocket_2.54mm:PinSocket_1x02_P2.54mm_Vertical, symbol Connector_Generic:Conn_01x02
- added J12, J3: Conn_01x04, Connector_PinSocket_1.27mm:PinSocket_1x04_P1.27mm_Vertical, symbol Connector_Generic:Conn_01x04
Connections:
- net GND: now also J12.4 (Pin_4), J3.4 (Pin_4)
- net HALL_MOTORA_A: now also J12.2 (Pin_2)
- net HALL_MOTORA_B: now also J12.3 (Pin_3)
- net HALL_MOTORB_A: now also J3.2 (Pin_2)
- net HALL_MOTORB_B: now also J3.3 (Pin_3)
- net MOTORA+: now also J11.1 (Pin_1)
- net MOTORA-: now also J11.2 (Pin_2)
- net MOTORB+: now also J2.1 (Pin_1)
- net MOTORB-: now also J2.2 (Pin_2)
- net +6V renamed +3V3
- net +3V3: now also J12.1 (Pin_1), J3.1 (Pin_1)
