File: PCB/MicroMouse/main_board/power_suply.kicad_sch (KiCad schematic)
At the start: 13 parts, among them U2 LT8608

Commit message: second PCB
Parts:
- removed C7: 100u, Capacitor_SMD:CP_Elec_6.3x7.7, symbol Device:C_Polarized
Connections:
- net +6V renamed +3V3
Other:
- note removed: "Prepocitat na 6V"

Commit message: PCB prototype
Parts:
- added J9: Conn_01x02, Connector_PinSocket_2.54mm:PinSocket_1x02_P2.54mm_Vertical, symbol Connector_Generic:Conn_01x02
Connections:
- net GND: now also J9.1 (Pin_1)
- net VCC: now also J9.2 (Pin_2)
Changed lines of the file:
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@@
+    )
+  )
+  (symbol (lib_id "power:GND") (at 139.7 39.37 0) (unit 1)
+    (in_bom yes) (on_board yes) (dnp no)
+    (property "Reference" "#PWR04" (at 139.7 45.72 0)
+      (effects (font (size 1.27 1.27)) hide)
+    )
+    (property "Value" "GND" (at 139.827 43.7642 0)
+      (effects (font (size 1.27 1.27)))
+    )
+    (property "Footprint" "" (at 139.7 39.37 0)
+      (effects (font (size 1.27 1.27)) hide)
+    )
+    (property "Datasheet" "" (at 139.7 39.37 0)
+      (effects (font (size 1.27 1.27)) hide)
+    )
+    (pin "1")
+    (instances
+      (project "main_board"
+        (path "/3863100a-f026-49db-8424-2d27c05016cc/112733e4-8eb6-414e-afb1-76d63d2a808b"
+          (reference "#PWR04") (unit 1)
+        )
+      )
     )
   )
@@
         )
       )
+    )
+  )
+  (symbol (lib_id "power:VCC") (at 139.7 36.83 0) (unit 1)
+    (in_bom yes) (on_board yes) (dnp no) (fields_autoplaced)
+    (property "Reference" "#PWR02" (at 139.7 40.64 0)
+      (effects (font (size 1.27 1.27)) hide)
+    )
+    (property "Value" "VCC" (at 139.7 31.75 0)
+      (effects (font (size 1.27 1.27)))
+    )
+    (property "Footprint" "" (at 139.7 36.83 0)
+      (effects (font (size 1.27 1.27)) hide)
+    )
+    (property "Datasheet" "" (at 139.7 36.83 0)
+      (effects (font (size 1.27 1.27)) hide)
+    )
+    (pin "1")
+    (instances
+      (project "main_board"
+        (path "/3863100a-f026-49db-8424-2d27c05016cc/112733e4-8eb6-414e-afb1-76d63d2a808b"
+          (reference "#PWR02") (unit 1)
+        )
+      )
+    )
+  )
+  (symbol (lib_id "Connector_Generic:Conn_01x02") (at 134.62 39.37 180) (unit 1)
+    (in_bom yes) (on_board yes) (dnp no) (fields_autoplaced)
+    (property "Reference" "J9" (at 134.62 30.48 0)
+      (effects (font (size 1.27 1.27)))
+    )
+    (property "Value" "Conn_01x02" (at 134.62 33.02 0)
+      (effects (font (size 1.27 1.27)))
+    )
+    (property "Footprint" "Connector_PinSocket_2.54mm:PinSocket_1x02_P2.54mm_Vertical" (at 134.62 39.37 0)
+      (effects (font (size 1.27 1.27)) hide)
+    )
+    (property "Datasheet" "~" (at 134.62 39.37 0)
+      (effects (font (size 1.27 1.27)) hide)
+    )
+    (pin "1")
+    (pin "2")
+    (instances
+      (project "main_board"
+        (path "/3863100a-f026-49db-8424-2d27c05016cc/112733e4-8eb6-414e-afb1-76d63d2a808b"
+          (reference "J9") (unit 1)
+        )
+      )
