File: PCB/MicroMouse/main_board/main_board.kicad_pcb (KiCad board)
At the start: 2 copper layers, 75 x 108.5 mm, 54 parts, among them J1 Conn_01x06, J10 Conn_01x05, J11 Conn_01x02, J12 Conn_01x04, J2 Conn_01x02, J3 Conn_01x04, J4 Conn_01x06, J5 Conn_01x06, J7 Conn_01x06, J8 Conn_01x06, J9 Conn_01x02, U2 LT8608, U3 TB6612FNG, U4 ESP32-WROOM-32U

Commit message: remove/rename var +png of tofs
Other:
- board text added: "++"
- board text added: "0"
- board text added: "100"
- board text added: "260"
- board text added: "315"
- board text added: "45"
- board text added: "<-- Y+"
- board text added: "^ | x+"

Commit message: angles in pcb
Other:
- board text added: "0 - 360"
- board text added: "TOF_1"
- board text added: "TOF_2"
- board text added: "TOF_3"
- board text added: "TOF_4"
