File: PCB/main_board/main_board.kicad_pcb (KiCad board)
At the start: 2 copper layers, 75 x 108.5 mm, 62 parts, among them J1 Conn_01x06, J13 Conn_01x06, J2 Conn_01x04, J4 Conn_01x06, J5 Conn_01x06, J6 Conn_01x06, J7 Conn_01x06, J8 Conn_01x06, J9 Conn_01x02, Q1 BSS138, Q2 BSS138, Q3 BSS138, Q4 BSS138, SW1 SW_Push, U1 LTC3525, U2 LT8608, U3 TB6612FNG, U4 ESP32-WROOM-32U

Commit message: edit board
Parts:
- removed H1, H14, H16, H2: MountingHole, MountingHole:MountingHole_2.7mm_M2.5_DIN965_Pad
- moved C5 22.2 mm to (136.1, 126.5)
- moved C1 22.2 mm to (131.1, 127.1)
- moved C2 22.2 mm to (133.5, 133.8)
- moved C3 22.2 mm to (123.0, 130.5)
- moved C6 22.2 mm to (114.3, 130.5)
- moved J9 22.2 mm to (109.3, 129.7)
- moved L1 22.2 mm to (136.1, 131.2)
- moved R2 22.2 mm to (123.0, 132.1)
- moved R3 22.2 mm to (123.0, 129.0)
- moved R4 22.2 mm to (123.0, 126.0)
- moved U2 22.2 mm to (128.8, 132.6)
- moved C4 22.2 mm to (123.0, 127.5)
- moved R1 22.2 mm to (129.6, 127.1)
Routing:
- net +3V3: track 340.9 -> 320.8 mm
- net VCC: track 116.8 -> 105.1 mm
- net GND: vias 378 -> 316
Other:
- board size 75 x 108.5 mm -> 75 x 87.8 mm
